Commit message: Add more links and joints

File: workspaces/whisky_bot_ws/src/whisky_bot_description/urdf/arm.xacro (robot description, xacro)
@@ -1,4 +1,5 @@
 <?xml version="1.0"?>
 <robot xmlns:xacro="http://www.ros.org/wiki/xacro">
+    <!-- links -->
     <link name="base_link">
         <visual>
@@ -24,5 +25,5 @@
                 <mesh filename="package://whisky_bot_description/meshes/type2.stl" scale="0.001 0.001 0.001"/>
             </geometry>
-            <origin xyz="-0.0125 -0.055 0" rpy="0 ${pi/2} 0"/>
+            <origin xyz="${-1*link_dim2/2} ${-1*link_dim1} 0" rpy="0 ${pi/2} 0"/>
             <material name="blue" />
         </visual>
@@ -31,5 +32,5 @@
         <visual>
             <geometry>
-                <cylinder length="0.052" radius="0.013"/>
+                <cylinder length="${link_dim1}" radius="0.013"/>
             </geometry>
             <origin xyz="0 0 0" rpy="0 ${pi/2} 0"/>
@@ -42,5 +43,5 @@
                 <mesh filename="package://whisky_bot_description/meshes/type2.stl" scale="0.001 0.001 0.001"/>
             </geometry>
-            <origin xyz="${-0.052/2} -0.055 -0.0125" rpy="0 0 0"/>
+            <origin xyz="${-1*link_dim3/2} ${-1*link_dim1} ${-1*link_dim2/2}" rpy="0 0 0"/>
             <material name="blue" />
         </visual>
@@ -51,5 +52,5 @@
                 <mesh filename="package://whisky_bot_description/meshes/type2.stl" scale="0.001 0.001 0.001"/>
             </geometry>
-            <origin xyz="${-0.052/2} 0.055 0.0125" rpy="${pi} 0 0"/>
+            <origin xyz="${-1*link_dim3/2} ${link_dim1} ${link_dim2/2}" rpy="${pi} 0 0"/>
             <material name="blue" />
         </visual>
@@ -58,8 +59,35 @@
         <visual>
             <geometry>
-                <box size="0.063 0.050 0.025"/>
+                <box size="${link_dim1} 0.050 ${link_dim2}"/>
             </geometry>
-            <origin xyz="0 -0.01 0" rpy="0 0 ${pi/2}"/>
+            <origin xyz="0 0 0" rpy="0 0 ${pi/2}"/>
             <material name="red" />
+        </visual>
+    </link>
+    <link name="link5">
+        <visual>
+            <geometry>
+                <mesh filename="package://whisky_bot_description/meshes/type2.stl" scale="0.001 0.001 0.001"/>
+            </geometry>
+            <origin xyz="${-1*link_dim1/2} ${1.3*link_dim1} ${link_dim2/2}" rpy="${pi} 0 0"/>
+            <material name="blue" />
+        </visual>
+    </link>
+    <link name="motor4">
+        <visual>
+            <geometry>
+                <box size="${link_dim1} 0.050 ${link_dim2}"/>
+            </geometry>
+            <origin xyz="0 0 0" rpy="0 0 ${pi/2}"/>
+            <material name="red" />
+        </visual>
+    </link>
+    <link name="link6">
+        <visual>
+            <geometry>
+                <mesh filename="package://whisky_bot_description/meshes/type2.stl" scale="0.001 0.001 0.001"/>
+            </geometry>
+            <origin xyz="${-1*link_dim1/2} ${-1*link_dim1/2} ${link_dim2/2}" rpy="${pi} 0 0"/>
+            <material name="blue" />
         </visual>
     </link>
@@ -68,5 +96,5 @@
         <parent link="base_link"/>
         <child link="link1"/>
-        <origin xyz="0.075 0.055 0.0475" rpy="0 0 0"/>
+        <origin xyz="0.075 ${link_dim1} 0.0475" rpy="0 0 0"/>
         <axis xyz="0 0 0"/>
     </joint>
@@ -81,5 +109,5 @@
         <parent link="link2"/>
         <child link="motor2"/>
-        <origin xyz="0 -0.025 0.0125" rpy="0 0 0"/>
+        <origin xyz="0 ${-1*link_dim2} ${link_dim2/2}" rpy="0 0 0"/>
         <axis xyz="0 0 0"/>
     </joint>
@@ -94,7 +122,5 @@
         <parent link="link3"/>
         <child link="link4"/>
-        <!-- <origin xyz="0 ${2*-0.055} 0" rpy="${pi} 0 0"/> -->
-        <!-- <origin xyz="${-0.052/2} -0.055 0" rpy="0 0 0"/> -->
-        <origin xyz="0 ${-2*0.055} 0" rpy="0 0 0"/>
+        <origin xyz="0 ${-2*link_dim1} 0" rpy="0 0 0"/>
     </joint>
     <joint name="joint6" type="revolute">
@@ -105,3 +131,22 @@
         <limit lower="-0.8" upper="${pi/2}" effort="1000.0" velocity="1.0"/>
     </joint>
+    <joint name="joint7" type="fixed">
+        <parent link="motor3"/>
+        <child link="link5"/>
+        <origin xyz="0 ${-2*link_dim1} 0" rpy="0 0 0"/>
+    </joint>
+    <joint name="joint8" type="revolute">
+        <parent link="link5"/>
+        <child link="motor4"/>
+        <origin xyz="0 ${link_dim2/2} 0" rpy="0 0 0"/>
+        <axis xyz="1 0 0"/>
+        <limit lower="${-pi/2}" upper="0.8" effort="1000.0" velocity="1.0"/>
+    </joint>
+    <joint name="joint9" type="revolute">
+        <parent link="motor4"/>
+        <child link="link6"/>
+        <origin xyz="0 0 0" rpy="0 0 0"/>
+        <axis xyz="0 1 0"/>
+        <limit lower="${-pi/2}" upper="0.8" effort="1000.0" velocity="1.0"/>
+    </joint>
 </robot>

File: workspaces/whisky_bot_ws/src/whisky_bot_description/urdf/common_properties.xacro (robot description, xacro)
@@ -1,4 +1,7 @@
 <?xml version="1.0"?>
 <robot xmlns:xacro="http://www.ros.org/wiki/xacro">
+    <xacro:property name="link_dim1" value="0.055" />
+    <xacro:property name="link_dim2" value="0.025" />
+    <xacro:property name="link_dim3" value="0.052" />
     <material name="grey">
         <color rgba="0.5 0.5 0.5 1"/>

Commit message: Add moveit2 configuration

File: workspaces/whisky_bot_ws/src/whisky_bot_description/urdf/arm.xacro (robot description, xacro)
@@ -19,4 +19,10 @@
             <material name="red" />
         </visual>
+        <collision>
+            <geometry>
+                <cylinder length="0.095" radius="0.004"/>
+            </geometry>
+            <origin xyz="0 0 0" rpy="0 0 0"/>
+        </collision>
     </link>
     <link name="link2">
@@ -28,4 +34,10 @@
             <material name="blue" />
         </visual>
+        <collision>
+            <geometry>
+                <mesh filename="package://whisky_bot_description/meshes/type2.stl" scale="0.001 0.001 0.001"/>
+            </geometry>
+            <origin xyz="${-1*link_dim2/2} ${-1*link_dim1} 0" rpy="0 ${pi/2} 0"/>
+        </collision>
     </link>
     <link name="motor2">
@@ -37,4 +49,10 @@
             <material name="red" />
         </visual>
+        <collision>
+            <geometry>
+                <cylinder length="${0.8*link_dim1}" radius="0.013"/>
+            </geometry>
+            <origin xyz="0 0 0" rpy="0 ${pi/2} 0"/>
+        </collision>
     </link>
     <link name="link3">
@@ -46,4 +64,10 @@
             <material name="blue" />
         </visual>
+        <collision>
+            <geometry>
+                <mesh filename="package://whisky_bot_description/meshes/type2.stl" scale="0.001 0.001 0.001"/>
+            </geometry>
+            <origin xyz="${-1*link_dim3/2} ${-1*link_dim1} ${-1*link_dim2/2}" rpy="0 0 0"/>
+        </collision>
     </link>
     <link name="link4">
@@ -55,4 +79,10 @@
             <material name="blue" />
         </visual>
+        <collision>
+            <geometry>
+                <mesh filename="package://whisky_bot_description/meshes/type2.stl" scale="0.001 0.001 0.001"/>
+            </geometry>
+            <origin xyz="${-1*link_dim3/2} ${link_dim1} ${link_dim2/2}" rpy="${pi} 0 0"/>
+        </collision>
     </link>
     <link name="motor3">
@@ -64,4 +94,10 @@
             <material name="red" />
         </visual>
+        <collision>
+            <geometry>
+                <box size="${link_dim1} ${0.8*0.050} ${link_dim2}"/>
+            </geometry>
+            <origin xyz="0 0 0" rpy="0 0 ${pi/2}"/>
+        </collision>
     </link>
     <link name="link5">
@@ -73,4 +109,10 @@
             <material name="blue" />
         </visual>
+        <collision>
+            <geometry>
+                <mesh filename="package://whisky_bot_description/meshes/type2.stl" scale="0.001 0.001 0.001"/>
+            </geometry>
+            <origin xyz="${-1*link_dim1/2} ${1.3*link_dim1} ${link_dim2/2}" rpy="${pi} 0 0"/>
+        </collision>
     </link>
     <link name="motor4">
@@ -82,4 +124,10 @@
             <material name="red" />
         </visual>
+        <collision>
+            <geometry>
+                <box size="${link_dim1} ${0.8*0.050} ${link_dim2}"/>
+            </geometry>
+            <origin xyz="0 0 0" rpy="0 0 ${pi/2}"/>
+        </collision>
     </link>
     <link name="link6">
@@ -91,4 +139,10 @@
             <material name="blue" />
         </visual>
+        <collision>
+            <geometry>
+                <mesh filename="package://whisky_bot_description/meshes/type2.stl" scale="0.001 0.001 0.001"/>
+            </geometry>
+            <origin xyz="${-1*link_dim1/2} ${-1*link_dim1/2} ${link_dim2/2}" rpy="${pi} 0 0"/>
+        </collision>
     </link>
     <!-- joints -->
